File: hardware/WOOTSwitch.kicad_pcb (KiCad board)
At the start: 2 copper layers, 100 x 88 mm, 133 parts, among them J1 Mini-DIN-4-G, J10 POWSEL, J11 TWI, J12 TWI, J13 Mini-DIN-4-G, J14 Mini-DIN-4-G, J15 Mini-DIN-4-G, J16 Mini-DIN-4-G, J2 Mini-DIN-4-G, J7 Barrel_Jack_MountingPin, J8 EXT_POW, J9 SW1, Q1 MMBT3904, Q11 2N7002, Q15 2N7002, Q17 2N7002, Q18 2N7002, Q19 2N7002, Q2 MMBT3904, Q20 2N7002, Q21 2N7002, Q22 2N7002, Q23 2N7002, Q24 2N7002, Q25 2N7002, Q26 2N7002, Q27 2N7002, Q28 2N7002, Q29 2N7002, Q3 MMBT3904, Q30 2N7002, Q31 2N7002, Q32 2N7002, Q33 2N7002, Q34 2N7002, Q35 2N7002, Q36 2N7002, Q37 2N7002, Q38 2N7002, Q39 2N7002, Q4 MMBT3904, Q40 2N7002, Q5 MMBT3904, Q6 MMBT3904, Q8 MMBT3904, Q9 2N7002, SW1 Switch1, U1 Pico, U2 LM1117-5.0

Commit message: Rebrand as WOOTSwitch
Parts:
- removed G***: LOGO, hootswitch:hootswitch
- removed SW1: Switch1, Button_Switch_THT:SW_SPST_Omron_B3F-315x_Angled
- added C15: 47uF, Capacitor_SMD:C_1206_3216Metric, F.Cu at (82.1, 105.8)
- added SW2: 1825910-6, hootswitch:SW_1825910-6-4, F.Cu at (154.2, 142.4)
- C1: value 100uF -> 47uF; footprint Capacitor_THT:CP_Radial_D6.3mm_P2.50mm -> Capacitor_SMD:C_1206_3216Metric
- moved R50 4.77 mm to (148.4, 140.8)
- moved C1 2.53 mm to (82.2, 103.4)
Routing:
- net GND: track 138.2 -> 164.2 mm, vias 86 -> 90
- net +3.3V: track 377.8 -> 371.3 mm, vias 4 -> 5
- net Net-(D7-A): track 40.5 -> 46.0 mm
- net Net-(U2-VI): track 11.9 -> 15.2 mm
- net /SWITCH: track 55.5 -> 52.5 mm
- net /C2_DO: track 40.1 -> 41.1 mm
- net /C1_DI: track 40.8 -> 40.2 mm
Other:
- board text added: "Licensed under CERN-OHL-S-2.0 github.com/Joes-Computer-Museum/WOOTSwitch"
- board text added: "{dblquote}hootswitch{dblquote} Originally by saybur This is WOOTSwitch, a hardware fork from Joe's Computer Museum Version: 2025.10"
- board text removed: "Licensed under CERN-OHL-S-2.0 github.com/TechByAndroda/hootswitch"
- board text removed: "Originally by saybur This is a hardware fork from: Tech by Androda, LLC Version: 2025.09"
- board text removed: "by saybur v2024a"
- board text removed: "{dblquote}hootswitch{dblquote}"
